Commit message: xiaoqiang gazebo

File: mygazebo/robots/myxiaoqiang/xiaoqiang_robot.xacro (robot description, xacro)
@@ -7,4 +7,5 @@
 <robot name="xiaoqiang_robot" xmlns:xacro="http://www.ros.org/wiki/xacro" >
   <xacro:include filename="$(find xiaoqiang_udrf)/robots/xiaoqiang.urdf.xacro"/>
+  <xacro:include filename="$(find mygazebo)/gazebo/xiaoqiang.gazebo" />
   <!-- <xacro:include filename="$(find mygazebo)/urdf/mycar_laser.urdf.xacro"/> -->
 <!--  <xacro:include filename="$(find mygazebo)/urdf/mycar_kinect.urdf.xacro"/>-->

File: ros_robot/xiaoqiang/xiaoqiang_udrf/robots/xiaoqiang.urdf.xacro (robot description, xacro)
@@ -6,12 +6,8 @@
 -->
 <robot name="xiaoqiang_urdf" xmlns:xacro="http://www.ros.org/wiki/xacro" >
-	<!-- <xacro:include filename="$(find mygazebo)/gazebo/mycar_base_gazebo.urdf.xacro"/>
-    <xacro:include filename="$(find mygazebo)/property/mycar_base_property.urdf.xacro"/> -->
-    <!-- <xacro:macro name="default_inertial" params="mass">
-    <inertial>
-      <mass value="${mass}" />
-      <inertia ixx="1.0" ixy="0.0" ixz="0.0" iyy="1.0" iyz="0.0" izz="1.0" />
-    </inertial>
-    </xacro:macro> -->
+  <xacro:arg name="robot_namespace" default=""/>
+  <xacro:property name="cameraSize" value="0.05"/>
+  <xacro:property name="cameraMass" value="0.1"/>
+  <xacro:property name="namespace" value="$(arg robot_namespace)" />
   <link
     name="base_link">

Commit message: xiaoqiang

File: mygazebo/robots/myxiaoqiang/xiaoqiang_robot.xacro (robot description, xacro)
@@ -7,4 +7,5 @@
 <robot name="xiaoqiang_robot" xmlns:xacro="http://www.ros.org/wiki/xacro" >
   <xacro:include filename="$(find xiaoqiang_udrf)/robots/xiaoqiang.urdf.xacro"/>
+  <!-- <xacro:include filename="$(find xiaoqiang_udrf)/robots/xiaoqiang_udrf.URDF"/> -->
   <xacro:include filename="$(find mygazebo)/gazebo/xiaoqiang.gazebo" />
   <!-- <xacro:include filename="$(find mygazebo)/urdf/mycar_laser.urdf.xacro"/> -->

File: ros_robot/xiaoqiang/xiaoqiang_udrf/robots/xiaoqiang.urdf.xacro (robot description, xacro)
@@ -15,7 +15,7 @@
       <origin
         xyz="-0.157602038251381 -0.00385000660473622 0.0465624701295276"
-        rpy="0 0 0" />
-      <mass
-        value="4.77346929236529" />
+        rpy="0 0.523 0" />
+      <mass
+        value="1.77346929236529" />
       <inertia
         ixx="0.0533752323010665"

File: ros_robot/xiaoqiang/xiaoqiang_udrf/robots/xiaoqiang_udrf.URDF (robot description, URDF)
Before this commit: robot xiaoqiang_udrf, 6 links, 5 joints
Joints:
- joint rot4: origin xyz=-0.258786796564404 6.46265772448196E-05 0.305000000000001 rpy=-1.5707963267949 -3.15213658012586E-15 -0.452067123629806 -> xyz=-0.258786796564404 6.46265772448196E-05 0.505000000000001 rpy=-1.5707963267949 -3.15213658012586E-15 -0.452067123629806
